File: PCB/Hackpad.kicad_sch (KiCad schematic)
At the start: 34 parts, among them SW13 RotaryEncoder_Switch, SW14 RotaryEncoder_Switch, U1 MOUDLE-SEEEDUINO-XIAO, U2 DM-OLED096-636, U3 MCP23017x-x-SP

Commit message: Apply minimal Blip PCB corrections
Parts:
- removed R3: 10k, symbol Device:R
- U1: value MOUDLE-SEEEDUINO-XIAO -> Seeed Studio XIAO ESP32-S3; footprint RF_Module:MCU_Seeed_ESP32C3 -> Blip:XIAO_ESP32S3_Socket; symbol XIAO_RP2040:MOUDLE-SEEEDUINO-XIAO -> Blip:XIAO_ESP32S3
Connections:
- net +3.3V: now also DS1.16 (~{RES}), DS1.4 (D/C/NC/SA0); no longer DS1.3 (REGVDD)
- net GND: now also DS1.10 (DB3/NC), DS1.11 (DB4/NC), DS1.12 (DB5/NC), DS1.13 (DB6/NC), DS1.14 (DB7/NC), DS1.3 (REGVDD), DS1.5 (R/W/NC), DS1.6 (E/NC)
- no-connect marks 23 -> 15
Changed lines of the file:
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@@
 	)
 	(no_connect
-		(at 176.53 121.92)
-	)
-	(no_connect
 		(at 245.11 115.57)
 	)
 	(no_connect
-		(at 176.53 129.54)
-	)
-	(no_connect
 		(at 270.51 135.89)
 	)
@@
 	)
 	(no_connect
-		(at 125.73 134.62)
-	)
-	(no_connect
 		(at 270.51 113.03)
 	)
@@
 	)
 	(no_connect
-		(at 176.53 124.46)
-	)
-	(no_connect
-		(at 176.53 132.08)
-	)
-	(no_connect
 		(at 212.09 62.23)
 	)
@@
 	)
 	(no_connect
-		(at 176.53 127)
-	)
-	(no_connect
-		(at 125.73 132.08)
-	)
-	(no_connect
 		(at 270.51 133.35)
 	)
@@
 	)
 	(no_connect
-		(at 125.73 129.54)
-	)
-	(no_connect
 		(at 270.51 138.43)
 	)
@@
 	(wire
 		(pts
-			(xy 125.73 114.3) (xy 119.38 114.3)
-		)
-		(stroke
-			(width 0)
-			(type default)
-		)
-	)
-	(wire
-		(pts
 			(xy 86.36 111.76) (xy 100.33 111.76)
 		)
@@
 	(wire
 		(pts
-			(xy 119.38 114.3) (xy 119.38 113.03)
-		)
-		(stroke
-			(width 0)
-			(type default)
-		)
-	)
-	(wire
-		(pts
 			(xy 76.2 69.85) (xy 76.2 87.63)
 		)
@@
 		)
 	)
+	(label "+3.3V"
+		(at 125.73 114.3 180)
+		(effects
+			(font (size 1.27 1.27))
+			(justify right bottom)
+		)
+	)
+	(label "+3.3V"
+		(at 125.73 132.08 180)
+		(effects
+			(font (size 1.27 1.27))
+			(justify right bottom)
+		)
+	)
+	(label "GND"
+		(at 125.73 129.54 180)
+		(effects
+			(font (size 1.27 1.27))
+			(justify right bottom)
+		)
+	)
+	(label "GND"
+		(at 125.73 134.62 180)
+		(effects
+			(font (size 1.27 1.27))
+			(justify right bottom)
+		)
+	)
+	(label "GND"
+		(at 176.53 121.92 0)
+		(effects (font (size 1.27 1.27)) (justify left bottom))
+	)
+	(label "GND"
+		(at 176.53 124.46 0)
+		(effects (font (size 1.27 1.27)) (justify left bottom))
+	)
+	(label "GND"
+		(at 176.53 127 0)
+		(effects (font (size 1.27 1.27)) (justify left bottom))
+	)
+	(label "GND"
+		(at 176.53 129.54 0)
+		(effects (font (size 1.27 1.27)) (justify left bottom))
+	)
+	(label "GND"
+		(at 176.53 132.08 0)
+		(effects (font (size 1.27 1.27)) (justify left bottom))
+	)
 	(label "SDA"
 		(at 176.53 116.84 0)
@@
 	)
 	(symbol
-		(lib_id "power:+3.3V")
+		(lib_id "power:GND")
 		(at 176.53 109.22 270)
 		(unit 1)
@@
 			)
 		)
-		(property "Value" "+3.3V"
+		(property "Value" "GND"
 			(at 180.34 109.2199 90)
 			(show_name no)
@@
 			)
 		)
-		(property "Description" "Power symbol creates a global label with name \"+3.3V\""
+		(property "Description" "Power symbol creates a global label with name \"GND\", ground"
 			(at 176.53 109.22 0)
 			(hide yes)
@@
 	)
 	(symbol
-		(lib_id "Device:R")
-		(at 119.38 109.22 0)
-		(unit 1)
-		(body_style 1)
-		(exclude_from_sim no)
-		(in_bom yes)
-		(on_board yes)
-		(in_pos_files yes)
-		(dnp no)
-		(fields_autoplaced yes)
-		(property "Reference" "R3"
-			(at 121.92 107.9499 0)
-			(show_name no)
-			(do_not_autoplace no)
-			(effects
-				(font
-					(size 1.27 1.27)
-				)
-				(justify left)
-			)
-		)
-		(property "Value" "10k"
-			(at 121.92 110.4899 0)
-			(show_name no)
-			(do_not_autoplace no)
-			(effects
-				(font
-					(size 1.27 1.27)
-				)
-				(justify left)
-			)
-		)
-		(property "Footprint" ""
-			(at 117.602 109.22 90)
-			(hide yes)
-			(show_name no)
-			(do_not_autoplace no)
-			(effects
-				(font
-					(size 1.27 1.27)
-				)
-			)
-		)
-		(property "Datasheet" ""
-			(at 119.38 109.22 0)
-			(hide yes)
-			(show_name no)
-			(do_not_autoplace no)
-			(effects
-				(font
-					(size 1.27 1.27)
-				)
-			)
-		)
-		(property "Description" "Resistor"
-			(at 119.38 109.22 0)
-			(hide yes)
-			(show_name no)
-			(do_not_autoplace no)
-			(effects
-				(font
-					(size 1.27 1.27)
-				)
-			)
-		)
-		(pin "1"
-		)
-		(pin "2"
-		)
-		(instances
-			(project "Hackpad"
-				(path "/b2ddfd41-41d8-40fc-950a-0913a8703706"
-					(reference "R3")
-					(unit 1)
-				)
-			)
-		)
-	)
-	(symbol
 		(lib_id "power:GND")
 		(at 176.53 137.16 90)
@@
 	)
 	(symbol
-		(lib_id "power:+3.3V")
-		(at 119.38 105.41 0)
-		(unit 1)
-		(body_style 1)
-		(exclude_from_sim no)
-		(in_bom yes)
-		(on_board yes)
-		(in_pos_files yes)
-		(dnp no)
-		(fields_autoplaced yes)
-		(property "Reference" "#PWR023"
-			(at 119.38 109.22 0)
-			(hide yes)
-			(show_name no)
-			(do_not_autoplace no)
-			(effects
-				(font
-					(size 1.27 1.27)
-				)
-			)
-		)
-		(property "Value" "+3.3V"
-			(at 119.38 100.33 0)
-			(show_name no)
-			(do_not_autoplace no)
-			(effects
-				(font
-					(size 1.27 1.27)
-				)
-			)
-		)
-		(property "Footprint" ""
-			(at 119.38 105.41 0)
-			(hide yes)
-			(show_name no)
-			(do_not_autoplace no)
-			(effects
-				(font
-					(size 1.27 1.27)
-				)
-			)
-		)
-		(property "Datasheet" ""
-			(at 119.38 105.41 0)
-			(hide yes)
-			(show_name no)
-			(do_not_autoplace no)
-			(effects
-				(font
-					(size 1.27 1.27)
-				)
-			)
-		)
-		(property "Description" "Power symbol creates a global label with name \"+3.3V\""
-			(at 119.38 105.41 0)
-			(hide yes)
-			(show_name no)
-			(do_not_autoplace no)
-			(effects
-				(font
-					(size 1.27 1.27)
-				)
-			)
-		)
-		(pin "1"
-		)
-		(instances
-			(project "Hackpad"
-				(path "/b2ddfd41-41d8-40fc-950a-0913a8703706"
-					(reference "#PWR023")
-					(unit 1)
-				)
-			)
-		)
-	)
-	(symbol
 		(lib_id "Switch:SW_Push")
 		(at 41.91 104.14 0)
@@
 	)
 	(symbol
-		(lib_id "XIAO_RP2040:MOUDLE-SEEEDUINO-XIAO")
+		(lib_id "Blip:XIAO_ESP32S3")
 		(at 231.14 54.61 0)
 		(unit 1)
@@
 			)
 		)
-		(property "Value" "MOUDLE-SEEEDUINO-XIAO"
+		(property "Value" "Seeed Studio XIAO ESP32-S3"
 			(at 232.41 41.91 0)
 			(show_name no)
@@
 			)
 		)
-		(property "Footprint" "RF_Module:MCU_Seeed_ESP32C3"
+		(property "Footprint" "Blip:XIAO_ESP32S3_Socket"
 			(at 214.63 52.07 0)
 			(hide yes)
@@
 			)
 		)
-		(property "Datasheet" ""
+		(property "Datasheet" "https://wiki.seeedstudio.com/xiao_esp32s3_getting_started/"
 			(at 214.63 52.07 0)
 			(hide yes)
