File: PCB/Hackpad.kicad_pcb (KiCad board)
At the start: 2 copper layers, 115.2 x 130.8 mm, 33 parts, among them SW13 RotaryEncoder_Switch, SW14 RotaryEncoder_Switch, U1 MOUDLE-SEEEDUINO-XIAO, U2 DM-OLED096-636, U3 MCP23017x-x-SP

Commit message: Apply minimal Blip PCB corrections
Parts:
- U1: value MOUDLE-SEEEDUINO-XIAO -> Seeed Studio XIAO ESP32-S3; footprint RF_Module:MCU_Seeed_ESP32C3 -> Blip:XIAO_ESP32S3_Socket
Connections:
- DS1 pad 10: unconnected-(DS1-DB3/NC-Pad10) -> GND
- DS1 pad 11: unconnected-(DS1-DB4/NC-Pad11) -> GND
- DS1 pad 12: unconnected-(DS1-DB5/NC-Pad12) -> GND
- DS1 pad 13: unconnected-(DS1-DB6/NC-Pad13) -> GND
- DS1 pad 14: unconnected-(DS1-DB7/NC-Pad14) -> GND
- DS1 pad 16: Net-(DS1-~{RES}) -> +3.3V
- DS1 pad 3: +3.3V -> GND
- DS1 pad 4: unconnected-(DS1-D/C/NC/SA0-Pad4) -> +3.3V
- DS1 pad 5: unconnected-(DS1-R/W/NC-Pad5) -> GND
- DS1 pad 6: unconnected-(DS1-E/NC-Pad6) -> GND
Routing:
- net GND: track 356.2 -> 414.1 mm
- net +3.3V: track 184.7 -> 208.9 mm

Commit message: Build Blip hardware validation gate
Routing:
- net /SDA: track 125.1 -> 175.7 mm, vias 3 -> 5
- net /ENC_D: track 85.7 -> 107.5 mm, vias 2 -> 1
- net GND: track 414.1 -> 415.0 mm
- net /ENC_SW: track 122.8 -> 123.6 mm
- net /SCL: track 123.2 -> 124.1 mm
- net /ENC_SW1: track 81.7 -> 80.8 mm
- net /ENC_A: track 135.9 -> 136.8 mm
- net +3.3V: track 208.9 -> 208.2 mm
- net /ENC_C: track 83.9 -> 83.4 mm
